File: field_eyes_v2.kicad_sch (KiCad schematic)
At the start: 156 parts, among them J101 SOLAR 6V, J201 PROG, J202 OLED, J203 DHT22, J301 U.FL LTE, J302 SIM holder (TE 2199337-5), J303 MODEM USB (DNP), J401 SMT100 (V+ GND A B), J402 7-in-1 NPK (V+ GND A B), J403 VALVE coil, Q101 AO3401A, Q102 AO3401A, Q103 2N7002, Q104 FS8205, Q105 AO3401A, Q106 2N7002, Q107 AO3401A, Q108 2N7002, Q201 MMBT3904, Q202 MMBT3904, Q301 MMBT3904, Q302 MMBT3904, Q303 MMBT3904, Q304 MMBT3904, Q305 MMBT3904, Q306 MMBT3904, Q401 MMBT3904, Q402 MMBT3904, SW201 RESET, SW202 BOOT, U101 CN3791, U102 DW01A, U103 XC6220B331MR, U104 MT3608, U201 ESP32-WROOM-32D, U301 A7672S, U302 SMF05C, U401 SP3485EN, U402 SP3485EN, U403 MX1508, U404 L78L09

Commit message: repositioned ccomponents
Parts:
- removed J201: PROG, Connector_PinHeader_2.54mm:PinHeader_1x06_P2.54mm_Vertical, symbol Connector_Generic:Conn_01x06
- removed J202: OLED, Connector_PinHeader_2.54mm:PinHeader_1x04_P2.54mm_Vertical, symbol Connector_Generic:Conn_01x04
- removed J203: DHT22, Connector_PinHeader_2.54mm:PinHeader_1x03_P2.54mm_Vertical, symbol Connector_Generic:Conn_01x03
- removed J401: SMT100 (V+ GND A B), TerminalBlock_Phoenix:TerminalBlock_Phoenix_PT-1,5-4-3.5-H_1x04_P3.50mm_Horizontal, symbol Connector:Screw_Terminal_01x04
- removed J402: 7-in-1 NPK (V+ GND A B), TerminalBlock_Phoenix:TerminalBlock_Phoenix_PT-1,5-4-3.5-H_1x04_P3.50mm_Horizontal, symbol Connector:Screw_Terminal_01x04
- removed U401, U402: SP3485EN, Package_SO:SOIC-8_3.9x4.9mm_P1.27mm, symbol Interface_UART:SP3485EN
- added C313: 33pF, Capacitor_SMD:C_0402_1005Metric, symbol Device:C
- added C408: 330nF 25V, Capacitor_SMD:C_0603_1608Metric, symbol Device:C
- added C409: 1uF, Capacitor_SMD:C_0603_1608Metric, symbol Device:C
- added J304: U.FL GPS, Connector_Coaxial:U.FL_Hirose_U.FL-R-SMT-1_Vertical, symbol Connector:Conn_Coaxial
- added L301: 56nH, Inductor_SMD:L_0805_2012Metric, symbol Device:L
- added R318: 0R, Resistor_SMD:R_0603_1608Metric, symbol Device:R
- added R319: 10k, Resistor_SMD:R_0603_1608Metric, symbol Device:R
- added R320, R321: 1k, Resistor_SMD:R_0603_1608Metric, symbol Device:R
- added R423, R425: 3.3k, Resistor_SMD:R_0603_1608Metric, symbol Device:R
- added R424, R426: 6.8k, Resistor_SMD:R_0603_1608Metric, symbol Device:R
- added SV1: PROG (as old SV1), field_eyes:MA03-2, symbol Connector_Generic:Conn_02x03_Odd_Even
- added U401, U402: MAX485ESA+T, Package_SO:SOIC-8_3.9x4.9mm_P1.27mm, symbol field_eyes:MAX485ESA+T
- added U405: L78L05, Package_TO_SOT_SMD:SOT-89-3, symbol Regulator_Linear:L78L05_SOT89
- added X1: 7-in-1 NPK (A B 12V GND), field_eyes:JST_XH_04_LongPad, symbol Connector_Generic:Conn_01x04
- added X2: SMT100 (A B 12V GND), field_eyes:JST_XH_04_LongPad, symbol Connector_Generic:Conn_01x04
- added X3: OLED (3V3 GND SDA SCL), field_eyes:JST_XH_04_LongPad, symbol Connector_Generic:Conn_01x04
- added X4: DHT22 (NC 3V3 DATA GND), field_eyes:JST_XH_04_LongPad, symbol Connector_Generic:Conn_01x04
Connections:
- net +12V_SENS: now also C408.1, U405.3 (IN), X1.3 (Pin_3), X2.3 (Pin_3)
- net +3V3: now also U301.P$116 (GNSS_VBKP), SV1.2 (Pin_2), X3.1 (Pin_1)
- net +3V3_SW: now also X4.2 (Pin_2); no longer C401.1, C402.1, R402.1, R403.1, R412.1, R413.1
- net DHT_DATA: now also X4.3 (Pin_3)
- net GND: now also C408.2, C409.2, J304.2 (Ext), R424.2, R426.2, SV1.6 (Pin_6), U401.5 (GND), U402.5 (GND), U405.2 (GND), X1.4 (Pin_4), X2.4 (Pin_4), X3.2 (Pin_2), X4.4 (Pin_4)
- net I2C_SCL: now also X3.4 (Pin_4)
- net I2C_SDA: now also X3.3 (Pin_3)
- net NPK_RX: now also R425.2, R426.1
- net NPK_TX: now also U402.4 (DI)
- net PROG_DTR: now also SV1.1 (Pin_1)
- net PROG_RTS: now also SV1.5 (Pin_5)
- net RS1_A: now also X2.1 (Pin_1)
- net RS1_AI: now also U401.6 (A)
- net RS1_B: now also X2.2 (Pin_2)
- net RS1_BI: now also U401.7 (B)
- net RS1_EN: now also U401.2 (~{RE}), U401.3 (DE)
- net RS2_A: now also X1.1 (Pin_1)
- net RS2_AI: now also U402.6 (A)
- net RS2_B: now also X1.2 (Pin_2)
- net RS2_BI: now also U402.7 (B)
- net RS2_EN: now also U402.2 (~{RE}), U402.3 (DE)
- net SMT_RX: now also R423.2, R424.1
- net SMT_TX: now also U401.4 (DI)
- net U0_RXD: now also SV1.4 (Pin_4)
- net U0_TXD: now also SV1.3 (Pin_3)
- net VDD_1V8: now also U301.P$97 (1V8_GNSS)
- new net +5V_SENS: C401.1, C402.1, C409.1, R402.1, R403.1, R412.1, R413.1, U401.8 (VCC), U402.8 (VCC), U405.1 (OUT)
- new net GNSS_PWRCTL: R319.1, U301.P$98 (GNSS_PWRCTL)
- new net GNSS_RXD: R320.1, U301.P$96 (GNSS_RXD)
- new net GNSS_TXD: R321.1, U301.P$95 (GNSS_TXD)
- new net GPS_ANT: C313.1, U301.P$90 (GPS_ANT)
- new net GPS_BIAS: L301.2, R318.1
- new net GPS_SIG: C313.2, J304.1 (In), L301.1
- new net MK_IN_3: R319.2, U301.P$20 (MK_IN_3)
- new net RS1_RO: R423.1, U401.1 (RO)
- new net RS2_RO: R425.1, U402.1 (RO)
- new net U3_RXD: R320.2, U301.P$49 (U3_RXD)
- new net U3_TXD: R321.2, U301.P$50 (U3_TXD)
- new net VDD_2V8: R318.2, U301.P$99 (VDD_2V8)
- no-connect marks 17 -> 18
Other:
- note added: "GPS ANTENNA (active antenna, as on the old board): the modem's 2.8 V feeds the antenna through R318 + L301 (56 nH); C313 blocks the DC. The built-in GNSS UART is linked to UART3 through R320/R321 and GNSS_PWRCTL goes to MK_IN_3 through R319 (SIMCom 3.11). 1V8_GNSS and GNSS_VBKP are powered. For a passive antenna, fit C313 only and do not fit R318/L301 (and send AT+CVAUXS=0)."
- note added: "MAX485ESA+T (the chip on the old board) on +5V_SENS, made by U405 (78L05) from the 12 V sensor rail, so it only has power while SENS_EN is on. RO swings 0-5 V: the 3.3k + 6.8k divider gives the ESP32 3.4 V (its pins are not 5 V tolerant). Direction is automatic: TX idle-high turns the MMBT3904 on and holds DE/RE low (receive); a 0 bit releases DE so the driver pulls the bus low; 1 bits come from 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"
- note added: "POWER TREE 6 V panel (1-2 W) -> CN3791 MPPT charger -> 18650 cell (DW01A/FS8205 protection) = VSYS 3.0-4.2 V VSYS -> A7672S VBAT directly (2 A bursts) VSYS -> XC6220 -> +3V3 (ESP32, always on) +3V3 -> AO3401A (SENS_EN) -> +3V3_SW (RS485, DHT22, NTC) VSYS -> AO3401A (SENS_EN) -> MT3608 -> +12V_SENS (soil sensors) -> 78L05 -> +5V_SENS (MAX485) and -> 78L09 -> 8.7 V valve reservoir (MX1508) WHAT CHA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"
- note removed: "POWER TREE 6 V panel (1-2 W) -> CN3791 MPPT charger -> 18650 cell (DW01A/FS8205 protection) = VSYS 3.0-4.2 V VSYS -> A7672S VBAT directly (2 A bursts) VSYS -> XC6220 -> +3V3 (ESP32, always on) +3V3 -> AO3401A (SENS_EN) -> +3V3_SW (RS485, DHT22, NTC) VSYS -> AO3401A (SENS_EN) -> MT3608 -> +12V_SENS (soil sensors) -> 78L09 -> 8.7 V valve reservoir (MX1508) WHAT CHANGED FROM THE OLD BOARD (security.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"
- note removed: "SP3485 (3.3 V, pin-compatible with MAX485) powered from +3V3_SW. Direction is automatic: TX idle-high turns the MMBT3904 on and holds DE/RE low (receive); a 0 bit releases DE so the driver pulls the bus low; 1 bits come from the 4.7k bias. 10 R + SM712 protect the field cable. 120 R termination not fitted (short cable, 9600 baud). Firmware: set the TX pins low/input before switching +3V3_SW off, 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"

Commit message: removed buttons
Parts:
- removed SW201: RESET, Button_Switch_SMD:SW_SPST_TL3342, symbol Switch:SW_Push
- removed SW202: BOOT, Button_Switch_SMD:SW_SPST_TL3342, symbol Switch:SW_Push
Changed lines of the file:
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@@
 	)
 	(text
-		"EN: 10k + 1 uF delay (Espressif reference) so the chip starts only after 3.3 V is stable.\nQ201/Q202: the usual two-transistor auto-reset, so esptool can reset and enter the bootloader through\nDTR/RTS of a USB-serial adapter (same pin order as the old SV1 header). Strapping pins IO0/IO2/IO12/IO15\nare left free or pulled the safe way. Flash pins (SD0-SD3, CLK, CMD) must stay unconnected.\nDo not connect the adapter's 3.3 V while the battery is fitted (two regulators would fight)."
+		"EN: 10k + 1 uF delay (Espressif reference) so the chip starts only after 3.3 V is stable.\nQ201/Q202: the usual two-transistor auto-reset, so esptool can reset and enter the bootloader through\nDTR/RTS of a USB-serial adapter (same pin order as the old SV1 header). Strapping pins IO0/IO2/IO12/IO15\nare left free or pulled the safe way. Flash pins (SD0-SD3, CLK, CMD) must stay unconnected.\nDo not connect the adapter's 3.3 V while the battery is fitted (two regulators would fight).\nThere are no reset or boot buttons: reset and boot mode come from the programming header SV1 (RTS -> EN, DTR -> IO0)."
 		(exclude_from_sim no)
 		(at 439.1 143.38 0)
@@
 	)
 	(symbol
-		(lib_id "Switch:SW_Push")
-		(at 459.74 213.36 90)
-		(unit 1)
-		(exclude_from_sim no)
-		(in_bom yes)
-		(on_board yes)
-		(dnp no)
-		(property "Reference" "SW201" (at 463.1 213.38 90) (effects (font (size 1.27 1.27)) (justify left)))
-		(property "Value" "RESET" (at 463.1 216.38 90) (effects (font (size 1.27 1.27)) (justify left)))
-		(property
-			"Footprint"
-			"Button_Switch_SMD:SW_SPST_TL3342"
-			(at 459.74 213.36 0)
-			(effects (font (size 1.27 1.27)) (hide yes))
-		)
-		(property "Datasheet" "~" (at 459.74 213.36 0) (effects (font (size 1.27 1.27)) (hide yes)))
-		(property "Description" "" (at 459.74 213.36 0) (effects (font (size 1.27 1.27)) (hide yes)))
-		(pin "1")
-		(pin "2")
-		(instances
-			(project "field_eyes_v2" (path "/1d2f7a40-5c1b-4f0e-9a6e-3b8c2d7e5f10" (reference "SW201") (unit 1)))
-		)
-	)
-	(wire
-		(pts (xy 459.74 218.44) (xy 459.74 220.98))
-		(stroke (width 0) (type default))
-	)
-	(symbol
-		(lib_id "power:GND")
-		(at 459.74 220.98 0)
-		(unit 1)
-		(exclude_from_sim no)
-		(in_bom no)
-		(on_board no)
-		(dnp no)
-		(property
-			"Reference"
-			"#PWR0038"
-			(at 464.82 219.71 0)
-			(effects (font (size 1.27 1.27)) (justify left) (hide yes))
-		)
-		(property "Value" "GND" (at 464.82 222.25 0) (effects (font (size 1.27 1.27)) (justify left) (hide yes)))
-		(property "Footprint" "" (at 459.74 220.98 0) (effects (font (size 1.27 1.27)) (hide yes)))
-		(property "Datasheet" "~" (at 459.74 220.98 0) (effects (font (size 1.27 1.27)) (hide yes)))
-		(property "Description" "" (at 459.74 220.98 0) (effects (font (size 1.27 1.27)) (hide yes)))
-		(pin "1")
-		(instances
-			(project "field_eyes_v2" (path "/1d2f7a40-5c1b-4f0e-9a6e-3b8c2d7e5f10" (reference "#PWR0038") (unit 1)))
-		)
-	)
-	(wire
-		(pts (xy 459.74 208.28) (xy 459.74 205.74))
-		(stroke (width 0) (type default))
-	)
-	(label
-		"ESP_EN"
-		(at 459.74 205.74 90)
-		(fields_autoplaced yes)
-		(effects (font (size 1.27 1.27)) (justify left bottom))
-	)
-	(symbol
-		(lib_id "Switch:SW_Push")
-		(at 459.74 254 90)
-		(unit 1)
-		(exclude_from_sim no)
-		(in_bom yes)
-		(on_board yes)
-		(dnp no)
-		(property "Reference" "SW202" (at 463.1 253.38 90) (effects (font (size 1.27 1.27)) (justify left)))
-		(property "Value" "BOOT" (at 463.1 256.38 90) (effects (font (size 1.27 1.27)) (justify left)))
-		(property
-			"Footprint"
-			"Button_Switch_SMD:SW_SPST_TL3342"
-			(at 459.74 254 0)
-			(effects (font (size 1.27 1.27)) (hide yes))
-		)
-		(property "Datasheet" "~" (at 459.74 254 0) (effects (font (size 1.27 1.27)) (hide yes)))
-		(property "Description" "" (at 459.74 254 0) (effects (font (size 1.27 1.27)) (hide yes)))
-		(pin "1")
-		(pin "2")
-		(instances
-			(project "field_eyes_v2" (path "/1d2f7a40-5c1b-4f0e-9a6e-3b8c2d7e5f10" (reference "SW202") (unit 1)))
-		)
-	)
-	(wire
-		(pts (xy 459.74 259.08) (xy 459.74 261.62))
-		(stroke (width 0) (type default))
-	)
-	(symbol
-		(lib_id "power:GND")
-		(at 459.74 261.62 0)
-		(unit 1)
-		(exclude_from_sim no)
-		(in_bom no)
-		(on_board no)
-		(dnp no)
-		(property
-			"Reference"
-			"#PWR0039"
-			(at 464.82 260.35 0)
-			(effects (font (size 1.27 1.27)) (justify left) (hide yes))
-		)
-		(property "Value" "GND" (at 464.82 262.89 0) (effects (font (size 1.27 1.27)) (justify left) (hide yes)))
-		(property "Footprint" "" (at 459.74 261.62 0) (effects (font (size 1.27 1.27)) (hide yes)))
-		(property "Datasheet" "~" (at 459.74 261.62 0) (effects (font (size 1.27 1.27)) (hide yes)))
-		(property "Description" "" (at 459.74 261.62 0) (effects (font (size 1.27 1.27)) (hide yes)))
-		(pin "1")
-		(instances
-			(project "field_eyes_v2" (path "/1d2f7a40-5c1b-4f0e-9a6e-3b8c2d7e5f10" (reference "#PWR0039") (unit 1)))
-		)
-	)
-	(wire
-		(pts (xy 459.74 248.92) (xy 459.74 246.38))
-		(stroke (width 0) (type default))
-	)
-	(label
-		"ESP_IO0"
-		(at 459.74 246.38 90)
-		(fields_autoplaced yes)
-		(effects (font (size 1.27 1.27)) (justify left bottom))
-	)
-	(symbol
